Commit message: Update

File: description/robot_core.xacro (robot description, xacro)
@@ -41,4 +41,7 @@
         </xacro:inertial_box>
     </link>
+    <gazebo reference="chassis">
+        <material>Gazebo/White</material>
+    </gazebo>
     <!-- LEFT FRONT WHEEL LINK -->
     <joint name="left_front_wheel_joint" type="continuous">
@@ -60,8 +63,13 @@
             </geometry>
         </collision>
-        <xacro:inertial_cylinder mass="0.1" length="0.045" radius="0.05">
+        <xacro:inertial_cylinder mass="0.25" length="0.045" radius="0.05">
             <origin xyz="0 0 0" rpy="0.0 0.0 0.0"/>
         </xacro:inertial_cylinder>
     </link>
+    <gazebo reference="left_front_wheel">
+        <material>Gazebo/Black</material>
+        <mu1 value="0.5"></mu1>
+        <mu2 value="0.4"></mu2>
+    </gazebo>
     <!-- LEFT REAR WHEEL LINK -->
     <joint name="left_rear_wheel_joint" type="continuous">
@@ -83,8 +91,13 @@
             </geometry>
         </collision>
-        <xacro:inertial_cylinder mass="0.1" length="0.045" radius="0.05">
+        <xacro:inertial_cylinder mass="0.25" length="0.045" radius="0.05">
             <origin xyz="0 0 0" rpy="0.0 0.0 0.0"/>
         </xacro:inertial_cylinder>
     </link>
+    <gazebo reference="left_rear_wheel">
+        <material>Gazebo/Black</material>
+        <mu1 value="0.5"></mu1>
+        <mu2 value="0.4"></mu2>
+    </gazebo>
     <!-- RIGHT FRONT WHEEL LINK -->
     <joint name="right_front_wheel_joint" type="continuous">
@@ -106,8 +119,13 @@
             </geometry>
         </collision>
-        <xacro:inertial_cylinder mass="0.1" length="0.045" radius="0.05">
+        <xacro:inertial_cylinder mass="0.25" length="0.045" radius="0.05">
             <origin xyz="0 0 0" rpy="0.0 0.0 0.0"/>
         </xacro:inertial_cylinder>
     </link>
+    <gazebo reference="right_front_wheel">
+        <material>Gazebo/Black</material>
+        <mu1 value="0.5"></mu1>
+        <mu2 value="0.4"></mu2>
+    </gazebo>
     <!-- RIGHT REAR WHEEL LINK -->
     <joint name="right_rear_wheel_joint" type="continuous">
@@ -129,7 +147,12 @@
             </geometry>
         </collision>
-        <xacro:inertial_cylinder mass="0.1" length="0.045" radius="0.05">
+        <xacro:inertial_cylinder mass="0.25" length="0.045" radius="0.05">
             <origin xyz="0 0 0" rpy="0.0 0.0 0.0"/>
         </xacro:inertial_cylinder>
     </link>
+    <gazebo reference="right_rear_wheel">
+        <material>Gazebo/Black</material>
+        <mu1 value="0.5"></mu1>
+        <mu2 value="0.4"></mu2>
+    </gazebo>
 </robot>
